Commit message: tweak: arm mount angle 45° → 90° (straight down)

File: archive/gibbonBot-RL/roarm_ws/roarm_description/ape.urdf (robot description, URDF)
Before this commit: robot ape_robot, 33 links, 32 joints
Joints:
- joint torso_to_bl_base_link: origin xyz=-0.12 0.10 -0.05 rpy=0 -0.785 0 -> xyz=-0.12 0.10 -0.05 rpy=0 -1.5708 0
- joint torso_to_br_base_link: origin xyz=-0.12 -0.10 -0.05 rpy=0 -0.785 0 -> xyz=-0.12 -0.10 -0.05 rpy=0 -1.5708 0
- joint torso_to_fl_base_link: origin xyz=0.12 0.10 -0.05 rpy=0 0.785 0 -> xyz=0.12 0.10 -0.05 rpy=0 1.5708 0
- joint torso_to_fr_base_link: origin xyz=0.12 -0.10 -0.05 rpy=0 0.785 0 -> xyz=0.12 -0.10 -0.05 rpy=0 1.5708 0

Commit message: fix: floor + gravity + freejoint + damping 2.0; add build_scene.py pipeline

File: archive/gibbonBot-RL/roarm_ws/roarm_description/ape.urdf (robot description, URDF)
Before this commit: robot ape_robot, 33 links, 32 joints
Links:
- added link world
Joints:
- added joint world_to_torso: type floating, parent world, child torso
