Commit message: RL training, GPU support, live multi-env viewer, physics tuning
- ape_env.py: Gymnasium env (63-dim obs, 24-dim action, reach-tree reward)
- train.py: PPO training via SB3, 8 envs, 10M steps, checkpoint + eval callbacks
- eval.py: headless evaluation, prints closest approach + success rate
- watch.py: persistent single-env viewer, hot-swaps policy on new checkpoint
- watch_multi.py: split-screen N-env viewer via mujoco.Renderer + OpenCV tiling
- Physics: torso mass 1→2 kg, kp 50→20, velocity penalty added to reward
- GPU: switched torch 2.11+cu130 → 2.5.1+cu121 (CUDA 12.2 driver compatible)
- Docs: README rewritten, DEVLOG updated, PLAN.md added for next steps

Co-Authored-By: Claude Sonnet 4.6 <noreply@anthropic.com>

File: archive/gibbonBot-RL/roarm_ws/roarm_description/ape.urdf (robot description, URDF)
Before this commit: robot ape_robot, 34 links, 33 joints
Links:
- link torso: mass 1.0 -> 2.0
